File: buck.kicad_sch (KiCad schematic)
At the start: 17 parts, among them IC5 LM5085MY_NOPB, Q12 PMOS

Commit message: LAYOUT IS GOINGGGG
Parts:
- removed Q12: PMOS, ExternalFootprints:SOIC127P600X175-8N, symbol Simulation_SPICE:PMOS
- added Q15: Si4463CDY, ExternalFootprints:SOIC127P600X175-8N, symbol utsvt-chips:SI7149ADP-T1-GE3
Connections:
- net ISEN: now also Q15.1 (S_1), Q15.2 (S_2), Q15.3 (S_3)
- net PGATE: now also Q15.4 (G)
- net at D13.1 (K), L1.1, R53.2: now also Q15.5 (D_1), Q15.6 (D_2), Q15.7 (D_3), Q15.8 (D_4)
Other:
- moved on the sheet: D13
