File: Cell-Characterization-Board.kicad_pcb (KiCad board)
At the start: 2 copper layers, 179 parts, among them IC1 MCP3304-CI_SL, IC2 INA4180A2IPWR, IC3 NCV8165ML330TCG, IC4 CYPD3177-24LQXQ, IC5 LM5085MY_NOPB, J1 USB_C_Receptacle_PowerOnly_6P, J2 USB_B_Micro, K1 V23105A5001A201, K2 V23105A5001A201, K3 V23105A5001A201, K4 V23105A5001A201, Q1 IRLML0030, Q10 IRLML0030, Q11 IRLML0030, Q12 PMOS, Q13 LRC L8050QLT1G, Q14 LRC L8050QLT1G, Q2 IRLML0030, Q3 IRLML0030, Q4 IRLML0030, Q5 IRLML0030, Q6 IRLML0030, Q7 IRF9358TRPBF, Q8 IRF9358TRPBF, Q9 BSL308PEH6327XTSA1, SW1 SW_Push, SW2 SW_Push, SW3 SW_Push, U2 ESP32-S3-WROOM-1, U3 MAX14611ETD+T, U4 CP2102N-A02-GQFN24

Commit message: LAYOUT IS GOINGGGG
Parts:
- removed Q12: PMOS, ExternalFootprints:SOIC127P600X175-8N
- removed U3: MAX14611ETD+T, Package_DFN_QFN:TDFN-14-1EP_3x3mm_P0.4mm_EP1.78x2.35mm
- added Q15: Si4463CDY, ExternalFootprints:SOIC127P600X175-8N, B.Cu at (150.5, 123.5)
- C10, C11, C12, C13, C14, C15, C16, C17, C18, C19, C20, C21, C22, C23, C24, C25, C26, C27, C28, C29, C3, C30, C31, C32, C33, C34, C35, C36, C37, C38, C39, C4, C40, C41, C5, C6, C7, C8, C9, D1, D10, D11, D12, D13, D2, D3, D4, D5, D6, D7, D8, D9, F1, F2, F3, F4, IC3, IC4, IC5, L1, Q1, Q10, Q11, Q13, Q14, Q2, Q3, Q4, Q5, Q6, Q7, Q8, Q9, R10, R11, R12, R13, R14, R15, R16, R17, R18, R19, R20, R21, R22, R23, R24, R25, R26, R27, R28, R29, R30, R31, R32, R33, R34, R35, R36, R37, R38, R39, R4, R40, R41, R42, R43, R44, R45, R46, R47, R48, R49, R5, R50, R51, R52, R53, R54, R55, R56, R57, R58, R59, R6, R60, R61, R7, R8, R9, RT1, RT2, RT3, RT4, TP12, TP13, TP14, TP15, TP16, TP17, TP7: moved to B.Cu
- U1, U2: moved to F.Cu
- moved K2 301.7 mm to (27.5, 130.3), turned to 90 degrees
- moved RT2 300.8 mm to (62.0, 122.8), turned to 180 degrees
- moved F2 295.9 mm to (68.5, 128.5), turned to 180 degrees
- moved D4 295.7 mm to (69.0, 132.8), turned to 180 degrees
- moved D5 295.6 mm to (69.0, 136.0), turned to 180 degrees
- moved R17 295.4 mm to (69.2, 139.2), turned to 180 degrees
- moved D6 290.3 mm to (77.0, 125.2), turned to 180 degrees
- moved Q4 288.7 mm to (79.8, 135.8), turned to 180 degrees
- moved Q3 288.6 mm to (79.8, 131.0), turned to 180 degrees
- moved TP3 287.3 mm to (119.8, 130.0)
- moved C11 286.2 mm to (84.2, 132.2), turned to 180 degrees
- moved C12 286.2 mm to (84.2, 135.2), turned to 180 degrees
- moved C8 286.0 mm to (84.2, 123.0), turned to 180 degrees
- moved C9 286.0 mm to (84.2, 126.0), turned to 180 degrees
- moved C10 286.0 mm to (84.2, 129.0), turned to 180 degrees
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Connections:
- C18 pad 1: Net-(IC3-GND_1) -> GND
- C20 pad 2: Net-(IC3-GND_2) -> GND
- IC3 pad 4: Net-(IC3-GND_1) -> GND
- IC3 pad 9: Net-(IC3-GND_2) -> GND
Routing:
- net Net-(U4-~{SUSPENDb}): track 22.0 -> 0.00 mm
- net Net-(U4-VBUS): track 20.3 -> 0.00 mm
- net Net-(IC4-CC2): track 14.3 -> 0.00 mm
- net Net-(D13-K): track 12.4 -> 0.00 mm
- net GND: track 11.7 -> 0.00 mm
- net /Power/VBUS_OUT: track 7.50 -> 0.00 mm
- net Net-(IC5-VCC): track 6.43 -> 0.00 mm
- net /Cell1/Batt-: track 2.42 -> 0.00 mm
- net /Cell1/Batt+: track 2.05 -> 0.00 mm
- net USB_MICRO_3V3: track 1.47 -> 0.00 mm
Other:
- board outline added: 165.2 x 113 mm
- board text added: "GND_IN"
- board text added: "Limit Resistors"
- board text added: "USB_FAULT"
- board text added: "VBUS_IN"

Commit message: cell layout plus rearranging
Parts:
- C1, C2, IC1, IC2, R1, R2, R3: moved to B.Cu
- RT4: moved to F.Cu
- moved K2 130.1 mm to (144.4, 73.3)
- moved K3 100.8 mm to (127.0, 89.0)
- moved K1 100.4 mm to (127.0, 68.2)
- moved K4 99.8 mm to (127.0, 47.5)
- moved D10 58.8 mm to (127.0, 50.8), turned to 0 degrees
- moved D11 58.8 mm to (127.0, 54.5), turned to 0 degrees
- moved Q10 48.7 mm to (127.5, 44.8), turned to -90 degrees
- moved R49 48.5 mm to (40.0, 52.0), turned to 0 degrees
- moved C30 40.0 mm to (43.8, 52.0), turned to 0 degrees
- moved R43 39.7 mm to (127.5, 40.5), turned to 0 degrees
- moved SW1 39.1 mm to (170.5, 53.5)
- moved R1 38.9 mm to (170.5, 54.5)
- moved C1 36.4 mm to (170.5, 52.5), turned to 180 degrees
- moved IC2 35.3 mm to (172.0, 80.5)
- moved R3 34.7 mm to (169.8, 69.8)
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Other:
- board text added: "+"
- board text added: "-"

Commit message: placement fini
Parts:
- RT1, RT2, RT3: moved to F.Cu
- moved D4 61.4 mm to (127.0, 112.8), turned to 0 degrees
- moved D5 61.1 mm to (127.0, 116.8), turned to 0 degrees
- moved D7 59.2 mm to (127.0, 92.2), turned to 0 degrees
- moved D8 59.1 mm to (127.0, 96.0), turned to 0 degrees
- moved D1 58.9 mm to (127.0, 71.2), turned to 0 degrees
- moved D2 58.9 mm to (127.0, 75.2), turned to 0 degrees
- moved Q3 53.2 mm to (127.5, 107.5), turned to -90 degrees
- moved Q5 50.7 mm to (127.8, 87.5), turned to -90 degrees
- moved R19 49.7 mm to (40.2, 130.0), turned to 0 degrees
- moved R27 49.7 mm to (40.2, 104.0), turned to 0 degrees
- moved Q1 49.4 mm to (127.2, 66.0), turned to -90 degrees
- moved R11 49.0 mm to (40.0, 78.0), turned to 0 degrees
- moved R13 45.2 mm to (127.8, 103.2), turned to 0 degrees
- moved R21 41.8 mm to (127.8, 83.0), turned to 0 degrees
- moved C17 40.7 mm to (44.0, 104.0), turned to 0 degrees
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Other:
- board size 165.2 x 113 mm -> 152.7 x 113 mm

Commit message: updated footprints and started tracing
Parts:
- added U3: MAX14611ETD+T, ExternalFootprints:MAX14611ETD_T, F.Cu at (148.2, 59.8)
- C24, C25: moved to F.Cu
- J1: value USB_C_Receptacle_PowerOnly_6P -> USB4125-GF-A-0190_REVA2; footprint Connector_USB:USB_C_Receptacle_HCTL_HC-TYPE-C-16P-01A -> ExternalFootprints:GCT_USB4125-GF-A-0190_REVA2
- moved R61 15.3 mm to (152.0, 41.8)
- moved IC1 12.6 mm to (152.2, 70.2), turned to 90 degrees
- moved R41 12.0 mm to (169.5, 106.2)
- moved Q14 10.1 mm to (152.8, 45.8)
- moved C2 8.90 mm to (142.3, 66.8), turned to 180 degrees
- moved R60 8.14 mm to (155.5, 45.8), turned to -90 degrees
- moved C1 6.86 mm to (163.8, 51.2)
- moved R1 6.86 mm to (163.8, 53.2)
- moved SW1 6.86 mm to (163.8, 52.2)
- moved IC2 4.62 mm to (142.3, 70.5)
- moved IC4 3.50 mm to (161.8, 100.8), turned to 45 degrees
- moved U1 2.70 mm to (157.8, 74.8)
- moved C25 2.54 mm to (174.0, 101.7)
- moved C24 2.40 mm to (171.0, 101.7)
- moved Q13 1.25 mm to (154.8, 41.8), turned to 90 degrees
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Routing:
- net /Cell1/Batt-: track 0.00 -> 96.5 mm
- net CURSET_1: track 0.00 -> 73.1 mm, vias 0 -> 3
- net EN: track 0.00 -> 35.2 mm, vias 0 -> 1
- net Net-(U4-VBUS): track 0.00 -> 27.0 mm, vias 0 -> 1
- net +3.3VA: track 0.00 -> 26.4 mm, vias 0 -> 4
- net /Cell1/REL_OUT: track 0.00 -> 24.3 mm
- net USB_D+: track 0.00 -> 22.6 mm
- net USB_D-: track 0.00 -> 22.4 mm
- net /Power/VBUS_OUT: track 0.00 -> 22.1 mm
- net USB_MICRO_3V3: track 0.00 -> 19.7 mm, vias 0 -> 1
- net /Power/VBUS_MIN: track 0.00 -> 19.1 mm
- net /Power/VBUS_MAX: track 0.00 -> 18.5 mm
- net Net-(Q8A-G): track 0.00 -> 17.9 mm
- net /Power/VBUS_IN: track 0.00 -> 17.5 mm
- net /Power/ISNK_COARSE: track 0.00 -> 17.2 mm
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- added copper zone on F.Cu, net GND
