File: Cell-Characterization-Board.kicad_sch (KiCad schematic)
At the start: 14 parts, among them IC1 MCP3304-CI_SL, IC2 INA4180A2IPWR, SW1 SW_Push, SW2 SW_Push, SW3 SW_Push, U2 ESP32-S3-WROOM-1, U3 MAX14611ETD+T

Commit message: updated footprints and started tracing
Parts:
- U3: footprint 21-0137_T1433+2C_MXM -> ExternalFootprints:MAX14611ETD_T
Changed lines of the file:
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@@
 			)
 		)
-		(property "Footprint" "21-0137_T1433+2C_MXM"
+		(property "Footprint" "ExternalFootprints:MAX14611ETD_T"
 			(at 81.28 127 0)
 			(effects
